Commit message: Updated joint angles based on Automata documentation

File: urdf/simpleEVA.urdf (robot description, URDF)
Before this commit: robot simpleEVA, 6 links, 5 joints
Joints:
- joint joint1: limit lower=-3.12413936107 upper=3.12413936107 effort=30 velocity=1.0 -> lower=-3.14159265359 upper=3.14159265359 effort=30 velocity=1.0
- joint joint2: limit lower=-2.70526034059 upper=1.2217304764 effort=30 velocity=1.0 -> lower=-2.77507351067 upper=1.29154364648 effort=30 velocity=1.0
- joint joint3: limit lower=-2.79252680319 upper=0.785398163397 effort=30 velocity=1.0 -> lower=-2.87979326579 upper=0.820304748437 effort=30 velocity=1.0
- joint joint4: limit lower=-3.12413936107 upper=3.12413936107 effort=30 velocity=1.0 -> lower=-3.14159265359 upper=3.14159265359 effort=30 velocity=1.0
- joint joint5: limit lower=-2.70526034059 upper=0.174532925199 effort=30 velocity=1.0 -> lower=-2.77507351067 upper=0.191986217719 effort=30 velocity=1.0

File: urdf/xacro/simpleEVA.urdf.xacro (robot description, xacro)
@@ -1,3 +1,4 @@
 <?xml version="1.0"?>
+<!-- Joint angles, link lengths and mass all found from Automata documentation -->
 <robot name="simpleEVA" xmlns:xacro="http://www.ros.org/wiki/xacro">
 	<!-- Import variables -->
@@ -14,5 +15,5 @@
 		<parent link="link1"/>
 		<child link="link2"/>
-		<xacro:jointLimits upper="179" lower="-179"/>
+		<xacro:jointLimits upper="180" lower="-180"/>
 		<axis xyz="0 0 1"/>
 		<origin xyz="0 0 ${l1_l}" rpy="0 0 0"/>
@@ -27,5 +28,5 @@
 		<parent link="link2"/>
 		<child link="link3"/>
-		<xacro:jointLimits upper="70" lower="-155"/>
+		<xacro:jointLimits upper="74" lower="-159"/>
 		<axis xyz="0 1 0"/>
 		<origin xyz="0 0 ${l2_l}" rpy="0 0 0"/>
@@ -40,5 +41,5 @@
 		<parent link="link3"/>
 		<child link="link4"/>
-		<xacro:jointLimits upper="45" lower="-160"/>
+		<xacro:jointLimits upper="47" lower="-165"/>
 		<axis xyz="0 1 0"/>
 		<origin xyz="0 0 ${l3_l}" rpy="0 0 0"/>
@@ -53,5 +54,5 @@
 		<parent link="link4"/>
 		<child link="link5"/>
-		<xacro:jointLimits upper="179" lower="-179"/>
+		<xacro:jointLimits upper="180" lower="-180"/>
 		<axis xyz="0 0 1"/>
 		<origin xyz="0 0 ${l4_l}" rpy="0 0 0"/>
@@ -66,5 +67,5 @@
 		<parent link="link5"/>
 		<child link="link6"/>
-		<xacro:jointLimits upper="10" lower="-155"/>
+		<xacro:jointLimits upper="11" lower="-159"/>
 		<axis xyz="0 1 0"/>
 		<origin xyz="0 0 ${l5_l}" rpy="0 0 0"/>

Commit message: Robot joints now have zero angle along x-axis

File: urdf/simpleEVA.urdf (robot description, URDF)
Before this commit: robot simpleEVA, 6 links, 5 joints
Joints:
- joint joint3: origin xyz=0 0 0.205 rpy=0 0 0 -> xyz=0.205 0 0 rpy=0 0 0
- joint joint4: axis 0 0 1 -> 1 0 0; origin xyz=0 0 0.124 rpy=0 0 0 -> xyz=0.124 0 0 rpy=0 0 0
- joint joint5: origin xyz=0 0 0.167 rpy=0 0 0 -> xyz=0.167 0 0 rpy=0 0 0

File: urdf/simpleEVA.urdf.xacro (robot description, xacro)
@@ -35,5 +35,5 @@
 	<link name="link3">
 		<xacro:cylinderInertial m="${m_total*(l3_l/l_total)}" l="${l3_l}" r="${l3_r}"/>
-		<xacro:cylinderGeometry name="link3" l="${l3_l}" r="${l3_r}" XYZ="0 ${-1*l3_r} ${l2_l}" RPY="0 0 0"/>
+		<xacro:cylinderGeometry name="link3" l="${l3_l}" r="${l3_r}" XYZ="${l3_l/2} ${-1*l3_r} 0" RPY="0 ${pi/2} 0"/>
 	</link>
 	<!-- 3rd joint -->
@@ -43,10 +43,10 @@
 		<xacro:jointLimits upper="47" lower="-165"/>
 		<axis xyz="0 1 0"/>
-		<origin xyz="0 0 ${l3_l}" rpy="0 0 0"/>
+		<origin xyz="${l3_l} 0 0" rpy="0 0 0"/>
 	</joint>
 	<!-- 4th link -->
 	<link name="link4">
 		<xacro:cylinderInertial m="${m_total*(l4_l/l_total)}" l="${l4_l}" r="${l4_r}"/>
-		<xacro:cylinderGeometry name="link4" l="${l4_l}" r="${l4_r}" XYZ="0 ${l4_r} ${l4_l/2}" RPY="0 0 0"/>
+		<xacro:cylinderGeometry name="link4" l="${l4_l}" r="${l4_r}" XYZ="${l4_l/2} ${l4_r} 0" RPY="0 ${pi/2} 0"/>
 	</link>
 	<!-- 4th joint -->
@@ -55,11 +55,11 @@
 		<child link="link5"/>
 		<xacro:jointLimits upper="180" lower="-180"/>
-		<axis xyz="0 0 1"/>
-		<origin xyz="0 0 ${l4_l}" rpy="0 0 0"/>
+		<axis xyz="1 0 0"/>
+		<origin xyz="${l4_l} 0 0" rpy="0 0 0"/>
 	</joint>
 	<!-- 5th link -->
 	<link name="link5">
 		<xacro:cylinderInertial m="${m_total*(l5_l/l_total)}" l="${l5_l}" r="${l5_r}"/>
-		<xacro:cylinderGeometry name="link5" l="${l5_l}" r="${l4_r}" XYZ="0 0 ${l5_l/2}" RPY="0 0 0"/>
+		<xacro:cylinderGeometry name="link5" l="${l5_l}" r="${l4_r}" XYZ="${l5_l/2} 0 0" RPY="0 ${pi/2} 0"/>
 	</link>
 	<!-- 5th joint -->
@@ -69,10 +69,15 @@
 		<xacro:jointLimits upper="11" lower="-159"/>
 		<axis xyz="0 1 0"/>
-		<origin xyz="0 0 ${l5_l}" rpy="0 0 0"/>
+		<origin xyz="${l5_l} 0 0" rpy="0 0 0"/>
 	</joint>
 	<!-- 6th link -->
 	<link name="link6">
 		<xacro:boxInertial m="${m_total*(l6_l/l_total)}" l="${l6_l}" d="${l6_d}" w="${l6_w}"/>
-		<xacro:boxGeometry name="link6" l="${l6_l}" d="${l6_d}" w="${l6_w}" XYZ="0 0 ${l6_l/2}" RPY="0 0 0"/>
+		<xacro:boxGeometry name="link6" l="${l6_l}" d="${l6_d}" w="${l6_w}" XYZ="${l6_l/2} 0 0" RPY="0 ${pi/2} 0"/>
 	</link>
+	<!-- Lamp -->
+	<!--<material name="yellow"
+	<link name="lamp">
+		<xacro:boxGeometry name="lamp" l="${lamp_l}" d="${lamp_d}" w="${lamp_w}" XYZ=
+	-->
 </robot>
