Commit message: Materials.xacro and lamp added to urdf

File: urdf/macros.xacro (robot description, xacro)
@@ -2,5 +2,5 @@
 <robot xmlns:xacro="http://wiki.ros.org/xacro">
 	<!-- Box geometry macro -->
-	<xacro:macro name="boxGeometry" params="name l d w XYZ RPY">
+	<xacro:macro name="boxGeometry" params="name l d w XYZ RPY colour">
 		<visual name="${name}Visual">
 			<geometry>
@@ -8,4 +8,5 @@
 			</geometry>
 			<origin xyz="${XYZ}" rpy="${RPY}"/>
+			<material name="${colour}"/>
 		</visual>
 		<collision name="${name}Collision">
@@ -17,5 +18,5 @@
 	</xacro:macro>
 	<!-- Cylinder geometry macro -->
-	<xacro:macro name="cylinderGeometry" params="name l r XYZ RPY">
+	<xacro:macro name="cylinderGeometry" params="name l r XYZ RPY colour">
 		<visual name="${name}Visual">
 			<geometry>
@@ -23,4 +24,5 @@
 			</geometry>
 			<origin xyz="${XYZ}" rpy="${RPY}"/>
+			<material name="${colour}"/>
 		</visual>
 		<collision name="${name}Collision">

File: urdf/simpleEVA.urdf (robot description, URDF)
Before this commit: robot simpleEVA, 6 links, 5 joints
Links:
- added link bulb; collision cylinder length=0.01 radius=0.015; visual cylinder length=0.01 radius=0.015
- added link controlBox; collision box size=0.075 0.11 0.078; visual box size=0.075 0.11 0.078
- added link lamp; collision box size=0.066 0.066 0.065; visual box size=0.066 0.066 0.065
Joints:
- added joint bulbToLamp: type fixed, parent lamp, child bulb
- added joint cBoxToLink1: type fixed, parent link1, child controlBox
- added joint joint6: type revolute, parent link6, child lamp, origin xyz=0.056 0 0.104 rpy=0 0 0, axis 0 0 1, limit lower=-3.12413936107 upper=3.12413936107 effort=30 velocity=1.0
- joint joint1: limit lower=-3.14159265359 upper=3.14159265359 effort=30 velocity=1.0 -> lower=-3.12413936107 upper=3.12413936107 effort=30 velocity=1.0
- joint joint2: limit lower=-2.77507351067 upper=1.29154364648 effort=30 velocity=1.0 -> lower=-2.70526034059 upper=1.2217304764 effort=30 velocity=1.0
- joint joint3: limit lower=-2.87979326579 upper=0.820304748437 effort=30 velocity=1.0 -> lower=-2.79252680319 upper=0.785398163397 effort=30 velocity=1.0; origin xyz=0.205 0 0 rpy=0 0 0 -> xyz=0 0 0.205 rpy=0 0 0
- joint joint4: axis 1 0 0 -> 0 0 1; limit lower=-3.14159265359 upper=3.14159265359 effort=30 velocity=1.0 -> lower=-3.12413936107 upper=3.12413936107 effort=30 velocity=1.0; origin xyz=0.124 0 0 rpy=0 0 0 -> xyz=0 0 0.124 rpy=0 0 0
- joint joint5: limit lower=-2.77507351067 upper=0.191986217719 effort=30 velocity=1.0 -> lower=-2.70526034059 upper=0.174532925199 effort=30 velocity=1.0; origin xyz=0.167 0 0 rpy=0 0 0 -> xyz=0 0 0.167 rpy=0 0 0

File: urdf/simpleEVA.urdf.xacro (robot description, xacro)
@@ -6,8 +6,10 @@
 	<!-- Import macros -->
 	<xacro:include filename="$(find simple_eva_description)/urdf/macros.xacro"/>
+	<!-- Import materials/colours -->
+	<xacro:include filename="$(find simple_eva_description)/urdf/materials.xacro"/>
 	<!-- 1st link -->
 	<link name="link1">
 		<xacro:boxInertial m="${m_total*(l1_l/l_total)}" l="${l1_l}" d="${l1_d}" w="${l1_w}"/>
-		<xacro:boxGeometry name="link1" l="${l1_l}" d="${l1_d}" w="${l1_w}" XYZ="0 0 ${l1_l/2}" RPY="0 0 0"/>
+		<xacro:boxGeometry name="link1" l="${l1_l}" d="${l1_d}" w="${l1_w}" XYZ="0 0 ${l1_l/2}" RPY="0 0 0" colour="offWhite"/>
 	</link>
 	<!-- 1st joint -->
@@ -15,12 +17,20 @@
 		<parent link="link1"/>
 		<child link="link2"/>
-		<xacro:jointLimits upper="180" lower="-180"/>
+		<xacro:jointLimits upper="179" lower="-179"/>
 		<axis xyz="0 0 1"/>
 		<origin xyz="0 0 ${l1_l}" rpy="0 0 0"/>
+	</joint>
+	<!-- "control box" -->
+	<link name="controlBox">
+		<xacro:boxGeometry name="controlBox" l="${cb_l}" w="${cb_w}" d="${cb_d}" XYZ="${l1_d/2} 0 ${cb_l/2}" RPY="0 0 0" colour="darkGrey"/>
+	</link>
+	<joint name="cBoxToLink1" type="fixed">
+		<parent link="link1"/>
+		<child link="controlBox"/>
 	</joint>
 	<!-- 2nd link -->
 	<link name="link2">
 		<xacro:cylinderInertial m="${m_total*(l2_l/l_total)}" l="${l2_l}" r="${l2_r}"/>
-		<xacro:cylinderGeometry name="link2" l="${l2_l}" r="${l2_r}" XYZ="0 ${l2_r} ${l2_l/2}" RPY="0 0 0"/>
+		<xacro:cylinderGeometry name="link2" l="${l2_l}" r="${l2_r}" XYZ="0 ${l2_r} ${l2_l/2}" RPY="0 0 0" colour="offWhite"/>
 	</link>
 	<!-- 2nd joint -->
@@ -28,5 +38,5 @@
 		<parent link="link2"/>
 		<child link="link3"/>
-		<xacro:jointLimits upper="74" lower="-159"/>
+		<xacro:jointLimits upper="70" lower="-155"/>
 		<axis xyz="0 1 0"/>
 		<origin xyz="0 0 ${l2_l}" rpy="0 0 0"/>
@@ -35,5 +45,5 @@
 	<link name="link3">
 		<xacro:cylinderInertial m="${m_total*(l3_l/l_total)}" l="${l3_l}" r="${l3_r}"/>
-		<xacro:cylinderGeometry name="link3" l="${l3_l}" r="${l3_r}" XYZ="${l3_l/2} ${-1*l3_r} 0" RPY="0 ${pi/2} 0"/>
+		<xacro:cylinderGeometry name="link3" l="${l3_l}" r="${l3_r}" XYZ="0 ${-1*l3_r} ${l2_l}" RPY="0 0 0" colour="offWhite"/>
 	</link>
 	<!-- 3rd joint -->
@@ -41,12 +51,12 @@
 		<parent link="link3"/>
 		<child link="link4"/>
-		<xacro:jointLimits upper="47" lower="-165"/>
+		<xacro:jointLimits upper="45" lower="-160"/>
 		<axis xyz="0 1 0"/>
-		<origin xyz="${l3_l} 0 0" rpy="0 0 0"/>
+		<origin xyz="0 0 ${l3_l}" rpy="0 0 0"/>
 	</joint>
 	<!-- 4th link -->
 	<link name="link4">
 		<xacro:cylinderInertial m="${m_total*(l4_l/l_total)}" l="${l4_l}" r="${l4_r}"/>
-		<xacro:cylinderGeometry name="link4" l="${l4_l}" r="${l4_r}" XYZ="${l4_l/2} ${l4_r} 0" RPY="0 ${pi/2} 0"/>
+		<xacro:cylinderGeometry name="link4" l="${l4_l}" r="${l4_r}" XYZ="0 ${l4_r} ${l4_l/2}" RPY="0 0 0" colour="offWhite"/>
 	</link>
 	<!-- 4th joint -->
@@ -54,12 +64,12 @@
 		<parent link="link4"/>
 		<child link="link5"/>
-		<xacro:jointLimits upper="180" lower="-180"/>
-		<axis xyz="1 0 0"/>
-		<origin xyz="${l4_l} 0 0" rpy="0 0 0"/>
+		<xacro:jointLimits upper="179" lower="-179"/>
+		<axis xyz="0 0 1"/>
+		<origin xyz="0 0 ${l4_l}" rpy="0 0 0"/>
 	</joint>
 	<!-- 5th link -->
 	<link name="link5">
 		<xacro:cylinderInertial m="${m_total*(l5_l/l_total)}" l="${l5_l}" r="${l5_r}"/>
-		<xacro:cylinderGeometry name="link5" l="${l5_l}" r="${l4_r}" XYZ="${l5_l/2} 0 0" RPY="0 ${pi/2} 0"/>
+		<xacro:cylinderGeometry name="link5" l="${l5_l}" r="${l4_r}" XYZ="0 0 ${l5_l/2}" RPY="0 0 0" colour="offWhite"/>
 	</link>
 	<!-- 5th joint -->
@@ -67,17 +77,32 @@
 		<parent link="link5"/>
 		<child link="link6"/>
-		<xacro:jointLimits upper="11" lower="-159"/>
+		<xacro:jointLimits upper="10" lower="-155"/>
 		<axis xyz="0 1 0"/>
-		<origin xyz="${l5_l} 0 0" rpy="0 0 0"/>
+		<origin xyz="0 0 ${l5_l}" rpy="0 0 0"/>
 	</joint>
 	<!-- 6th link -->
 	<link name="link6">
 		<xacro:boxInertial m="${m_total*(l6_l/l_total)}" l="${l6_l}" d="${l6_d}" w="${l6_w}"/>
-		<xacro:boxGeometry name="link6" l="${l6_l}" d="${l6_d}" w="${l6_w}" XYZ="${l6_l/2} 0 0" RPY="0 ${pi/2} 0"/>
+		<xacro:boxGeometry name="link6" l="${l6_l}" d="${l6_d}" w="${l6_w}" XYZ="${l5_r} 0 ${l6_d}" RPY="0 0 0" colour="offWhite"/>
 	</link>
+	<!-- 6th joint -->
+	<joint name="joint6" type="revolute">
+		<parent link="link6"/>
+		<child link="lamp"/>
+		<xacro:jointLimits upper="179" lower="-179"/>
+		<axis xyz="0 0 1"/>
+		<origin xyz="${l5_r} 0 ${l6_l}" rpy="0 0 0"/>
+	</joint>
 	<!-- Lamp -->
-	<!--<material name="yellow"
 	<link name="lamp">
-		<xacro:boxGeometry name="lamp" l="${lamp_l}" d="${lamp_d}" w="${lamp_w}" XYZ=
-	-->
+		<xacro:boxGeometry name="lamp" l="${lamp_l}" d="${lamp_d}" w="${lamp_w}" XYZ="0 0 ${lamp_l/2}" RPY="0 0 0" colour="black"/>
+	</link>
+	<!-- "bulb" -->
+	<link name="bulb">
+		<xacro:cylinderGeometry name="bulb" l="${bulb_l}" r="${bulb_r}" XYZ="0 0 ${lamp_l-(bulb_l/2)}" RPY="0 0 0" colour="yellow"/>
+	</link>
+	<joint name="bulbToLamp" type="fixed">
+		<parent link="lamp"/>
+		<child link="bulb"/>
+	</joint>
 </robot>

File: urdf/variables.xacro (robot description, xacro)
@@ -28,3 +28,10 @@
 	<xacro:property name="lamp_w" value="0.066"/>
 	<xacro:property name="lamp_d" value="0.066"/>
+	<!-- "control box" variables -->
+	<xacro:property name="cb_l" value="0.078"/>
+	<xacro:property name="cb_d" value="0.075"/>
+	<xacro:property name="cb_w" value="0.110"/>
+	<!-- "bulb" variables -->
+	<xacro:property name="bulb_l" value="0.010"/>
+	<xacro:property name="bulb_r" value="0.015"/>
 </robot>
